File: amp.kicad_sch (KiCad schematic)
At the start: 92 parts, among them J1 Input a/b/M, J3 Speaker 8/6/4/0, P1 25k, P2 25k, P3 25k, P4 25k, P5 25k, P6 25k, T1 E-1220, T2 OPT PPP Rkk 330R

Commit message: Fix bias pot wiring: grid leak resistors to pot wiper
R19..R24 now connect to the wiper (pin 2) of P1..P6; the pots form the
divider between the 33k resistors and the bias line.

Co-Authored-By: Claude Opus 5.5 <noreply@anthropic.com>
Parts:
- removed C10: 22µ/100V, Capacitor_THT:CP_Radial_D8.0mm_P3.50mm, symbol Device:C_Polarized
- removed C4: 47µ/450V, Capacitor_THT:CP_Radial_D18.0mm_P7.50mm, symbol Device:C_Polarized
- removed C6: 3.3p, Capacitor_THT:C_Disc_D5.0mm_W2.5mm_P5.00mm, symbol Device:C
- removed P1: 25k, Potentiometer_THT:Potentiometer_Piher_PT-10-V10_Vertical_Hole, symbol Device:R_Potentiometer_Trim
- removed R10: 220k, Resistor_THT:R_Axial_DIN0207_L6.3mm_D2.5mm_P10.16mm_Horizontal, symbol Device:R
- removed R14: 33k, Resistor_THT:R_Axial_DIN0207_L6.3mm_D2.5mm_P10.16mm_Horizontal, symbol Device:R
- removed R16: 10k, Resistor_THT:R_Axial_DIN0414_L11.9mm_D4.5mm_P15.24mm_Horizontal, symbol Device:R
- removed R4: 150k, Resistor_THT:R_Axial_DIN0207_L6.3mm_D2.5mm_P10.16mm_Horizontal, symbol Device:R
- removed R49, R50: 47R, Resistor_THT:R_Axial_DIN0207_L6.3mm_D2.5mm_P10.16mm_Horizontal, symbol Device:R
- removed R5: 2.7k, Resistor_THT:R_Axial_DIN0414_L11.9mm_D4.5mm_P15.24mm_Horizontal, symbol Device:R
- removed unit 1 of V1
- removed unit 1 of V2
- removed unit 1 of V3
- removed unit 2 of V4
- added C1: 2.2µ/40V bip., Capacitor_THT:CP_Radial_D6.3mm_P2.50mm, symbol Device:C
- added C16, C18: 47µ/100V, Capacitor_THT:CP_Radial_D10.0mm_P5.00mm, symbol Device:C_Polarized
- added D2, D3: 100V, Diode_THT:D_DO-41_SOD81_P10.16mm_Horizontal, symbol Device:D_Zener
- added D5: 1N4007, Diode_THT:D_DO-41_SOD81_P10.16mm_Horizontal, symbol Device:D
- added J3: Speaker 8/6/4/0, TerminalBlock_Phoenix:TerminalBlock_Phoenix_MKDS-1,5-4_1x04_P5.00mm_Horizontal, symbol Connector_Generic:Conn_01x04
- added R15: 10k, Resistor_THT:R_Axial_DIN0414_L11.9mm_D4.5mm_P15.24mm_Horizontal, symbol Device:R
- added R18: 6.8k, Resistor_THT:R_Axial_DIN0207_L6.3mm_D2.5mm_P10.16mm_Horizontal, symbol Device:R
- added R2: 68k, Resistor_THT:R_Axial_DIN0207_L6.3mm_D2.5mm_P10.16mm_Horizontal, symbol Device:R
- added R3: 2.2k, Resistor_THT:R_Axial_DIN0207_L6.3mm_D2.5mm_P10.16mm_Horizontal, symbol Device:R
- added R7: 1M, Resistor_THT:R_Axial_DIN0207_L6.3mm_D2.5mm_P10.16mm_Horizontal, symbol Device:R
- added R8: 2.7k, Resistor_THT:R_Axial_DIN0207_L6.3mm_D2.5mm_P10.16mm_Horizontal, symbol Device:R
- added R9: 47k, Resistor_THT:R_Axial_DIN0207_L6.3mm_D2.5mm_P10.16mm_Horizontal, symbol Device:R
- added T1: E-1220, symbol ppp:T_Input_Shield
- C10: renamed from D3; value 100V -> 22µ/100V; footprint Diode_THT:D_DO-41_SOD81_P10.16mm_Horizontal -> Capacitor_THT:CP_Radial_D8.0mm_P3.50mm; symbol Device:D_Zener -> Device:C_Polarized
- C4: renamed from R2; value 68k -> 47µ/450V; footprint Resistor_THT:R_Axial_DIN0207_L6.3mm_D2.5mm_P10.16mm_Horizontal -> Capacitor_THT:CP_Radial_D18.0mm_P7.50mm; symbol Device:R -> Device:C_Polarized
- C6: renamed from C18; value 47µ/100V -> 3.3p; footprint Capacitor_THT:CP_Radial_D10.0mm_P5.00mm -> Capacitor_THT:C_Disc_D5.0mm_W2.5mm_P5.00mm; symbol Device:C_Polarized -> Device:C
- P1: renamed from R15; value 10k -> 25k; footprint Resistor_THT:R_Axial_DIN0414_L11.9mm_D4.5mm_P15.24mm_Horizontal -> Potentiometer_THT:Potentiometer_Piher_PT-10-V10_Vertical_Hole; symbol Device:R -> Device:R_Potentiometer_Trim
- R10: renamed from D5; value 1N4007 -> 220k; footprint Diode_THT:D_DO-41_SOD81_P10.16mm_Horizontal -> Resistor_THT:R_Axial_DIN0207_L6.3mm_D2.5mm_P10.16mm_Horizontal; symbol Device:D -> Device:R
- R11: renamed from R7; value 1M -> 47k; footprint Resistor_THT:R_Axial_DIN0207_L6.3mm_D2.5mm_P10.16mm_Horizontal -> Resistor_THT:R_Axial_DIN0414_L11.9mm_D4.5mm_P15.24mm_Horizontal
- R12: renamed from R8; value 2.7k -> 47k; footprint Resistor_THT:R_Axial_DIN0207_L6.3mm_D2.5mm_P10.16mm_Horizontal -> Resistor_THT:R_Axial_DIN0414_L11.9mm_D4.5mm_P15.24mm_Horizontal
- R14: renamed from D2; value 100V -> 33k; footprint Diode_THT:D_DO-41_SOD81_P10.16mm_Horizontal -> Resistor_THT:R_Axial_DIN0207_L6.3mm_D2.5mm_P10.16mm_Horizontal; symbol Device:D_Zener -> Device:R
- R16: renamed from R11; value 47k -> 10k
- R4: renamed from C1; value 2.2µ/40V bip. -> 150k; footprint Capacitor_THT:CP_Radial_D6.3mm_P2.50mm -> Resistor_THT:R_Axial_DIN0207_L6.3mm_D2.5mm_P10.16mm_Horizontal; symbol Device:C -> Device:R
- R49: renamed from C16; value 47µ/100V -> 47R; footprint Capacitor_THT:CP_Radial_D10.0mm_P5.00mm -> Resistor_THT:R_Axial_DIN0207_L6.3mm_D2.5mm_P10.16mm_Horizontal; symbol Device:C_Polarized -> Device:R
- R5: renamed from R3; value 2.2k -> 2.7k; footprint Resistor_THT:R_Axial_DIN0207_L6.3mm_D2.5mm_P10.16mm_Horizontal -> Resistor_THT:R_Axial_DIN0414_L11.9mm_D4.5mm_P15.24mm_Horizontal
- R50: renamed from R18; value 6.8k -> 47R
- V1: renamed from T1; value E-1220 -> ECC83; footprint (none) -> Valve:Valve_Noval_P; symbol ppp:T_Input_Shield -> Valve:ECC83
- V2: renamed from R9; value 47k -> ECC81; footprint Resistor_THT:R_Axial_DIN0207_L6.3mm_D2.5mm_P10.16mm_Horizontal -> Valve:Valve_Noval_P; symbol Device:R -> Valve:ECC81
- V3: renamed from R12; value 47k -> EL34; footprint Resistor_THT:R_Axial_DIN0414_L11.9mm_D4.5mm_P15.24mm_Horizontal -> Valve:Valve_Octal; symbol Device:R -> ppp:EL34
- V4: renamed from J3; value Speaker 8/6/4/0 -> EL34; footprint TerminalBlock_Phoenix:TerminalBlock_Phoenix_MKDS-1,5-4_1x04_P5.00mm_Horizontal -> Valve:Valve_Octal; symbol Connector_Generic:Conn_01x04 -> ppp:EL34
Connections:
- net A1: now also V3.3 (A)
- net G1: now also R11.2, R15.1; no longer P1.1, R16.2
- net G2: now also R12.2, R16.2; no longer V3.2
- net GND: now also C10.2, R49.2, R50.1, R2.2, R9.2, T1.4 (S2), T1.5 (SH); no longer V1.4 (S2), V1.5 (SH), V2.2
- net HEATER_A: now also R49.1, V4.2 (F1)
- net HEATER_B: now also R50.2, V4.7 (F2)
- net M2: now also C16.1, C18.1; no longer C6.1, R49.1
- net UG1: now also D5.1 (K); no longer R10.1 (K)
- net at C15.2, R17.2: now also D5.2 (A); no longer R10.2 (A)
- net at P3.1, R27.2: no longer R21.2
- net at V2.2 (G): now also C10.1, R14.2
- net at C11.1, C13.1, C8.1: now also V2.6 (A), R15.2; no longer P1.2
- net at C5.1, D1.1 (K), V1.1 (A): now also R11.1, R12.1, R5.2; no longer R16.1, V3.1
- net at V1.3 (K): now also R8.1; no longer R12.1
- net at C7.2, V1.2 (G): now also R7.1; no longer R11.1
- net at R13.1, V2.3 (K): now also V2.8 (K)
- net at P6.3, R30.1: no longer R24.1
- net at C2.2, C3.1: now also V1.7 (G), R3.2; no longer R5.2
- net at P5.1, R29.2: no longer R23.2
- net at D4.1 (K): now also D3.2 (A); no longer C10.2 (A)
- net at C12.2, C14.2, C9.2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: now also R16.1
- net at R25.2: now also P1.1; no longer R19.2
- net at C17.2, P3.3, P5.3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: now also P1.3; no longer P3.2, P5.2
- net at T2.4 (8): now also J3.1 (Pin_1); no longer V4.1 (Pin_1)
- net at T2.5 (6): now also J3.2 (Pin_2); no longer V4.2 (Pin_2)
- net at T2.6 (4): now also J3.3 (Pin_3); no longer V4.3 (Pin_3)
- net at T2.7 (0): now also J3.4 (Pin_4); no longer V4.4 (Pin_4)
- net at P4.3, R28.1: no longer R22.1
- net at D1.2 (A): now also D2.1 (K); no longer R14.1 (K)
- net at P2.3, R26.1: no longer R20.1
- net at R31.2: now also V3.5 (G1)
- net at J1.1 (Pin_1): now also T1.1 (a); no longer V1.1 (a)
- net at J1.2 (Pin_2): now also T1.2 (b); no longer V1.2 (b)
- net at R6.1: now also C6.1, R10.1, V1.8 (K)
- net at R37.1: now also C6.2, R10.2, V3.1 (G3), V3.8 (K)
- net at C2.1, C7.1: now also R4.2, V1.6 (A)
- net at C4.1, R5.1: now also R4.1; no longer R4.2
- net at R43.2: now also V3.4 (G2)
- new net: P2.2, R20.1
- new net: P1.2, R19.2
- new net: P6.2, R24.1
- new net: P3.2, R21.2
- new net: P5.2, R23.2
- new net: C18.2, P2.1, P4.1, P6.1, R18.1
- new net: P4.2, R22.1
- new net: D2.2 (A), D3.1 (K)
- new net: R14.1, R7.2, R8.2, R9.1, V2.7 (G)
- new net: C1.2, R2.1, R3.1
- new net: C16.2, D6.2 (A), R18.2
- new net: C1.1, R1.1, T1.3 (S1)
Other:
- moved on the sheet: R11, R12, R16, R5, R50

Commit message: Add AP-634/2 output transformer data to T2
Value AP-634/2 (EXPERIENCE electronics), Rkk 330 Ohm / >140 W shown on
the sheet; manufacturer, MPN, secondary taps, core and frequency
response as symbol fields. Project file expanded to KiCad defaults.

Co-Authored-By: Claude Opus 5.5 <noreply@anthropic.com>
Parts:
- T2: value OPT PPP Rkk 330R -> AP-634/2; Core (none) -> MD 85 B, 85 x 102 x 75 mm, stud mounting; Frequency response (none) -> 20 Hz...20 kHz (-0.3 dB), 80 kHz (-3 dB); MPN (none) -> AP-634/2; Manufacturer (none) -> EXPERIENCE electronics; Secondary (none) -> 4 / 6 / 8 Ohm; Specs (none) -> Rkk 330Ω, >140W
Other:
- note added: "Original designators: V1=Rö1 (ECC83), V2=Rö2 (ECC81), V3..V8=Rö3..Rö8 (EL34), T1=Ü1 (E-1220), T2=Ü2 (AP-634/2). Supply rails A1/G1/M1, A2/G2/M2 and UG1/UG2 come from the power supply sheet. Upper tubes: anode A1, screen G1, cathode M1 (G1 is referenced to M1). Lower tubes: anode A2, screen G2, cathode M2 (G2 is referenced to M2). Ug1/Ug2: bias windings, floating on M1/M2; bias adjust P1..P6."
- note removed: "Original designators: V1=Rö1 (ECC83), V2=Rö2 (ECC81), V3..V8=Rö3..Rö8 (EL34), T1=Ü1 (E-1220), T2=Ü2. Supply rails A1/G1/M1, A2/G2/M2 and UG1/UG2 come from the power supply sheet. Upper tubes: anode A1, screen G1, cathode M1 (G1 is referenced to M1). Lower tubes: anode A2, screen G2, cathode M2 (G2 is referenced to M2). Ug1/Ug2: bias windings, floating on M1/M2; bias adjust P1..P6."
Changed lines of the file:
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@@
 		)
 	)
-	(text "Original designators: V1=Rö1 (ECC83), V2=Rö2 (ECC81), V3..V8=Rö3..Rö8 (EL34), T1=Ü1 (E-1220), T2=Ü2.\nSupply rails A1/G1/M1, A2/G2/M2 and UG1/UG2 come from the power supply sheet.\nUpper tubes: anode A1, screen G1, cathode M1 (G1 is referenced to M1).\nLower tubes: anode A2, screen G2, cathode M2 (G2 is referenced to M2).\nUg1/Ug2: bias windings, floating on M1/M2; bias adjust P1..P6."
+	(text "Original designators: V1=Rö1 (ECC83), V2=Rö2 (ECC81), V3..V8=Rö3..Rö8 (EL34), T1=Ü1 (E-1220), T2=Ü2 (AP-634/2).\nSupply rails A1/G1/M1, A2/G2/M2 and UG1/UG2 come from the power supply sheet.\nUpper tubes: anode A1, screen G1, cathode M1 (G1 is referenced to M1).\nLower tubes: anode A2, screen G2, cathode M2 (G2 is referenced to M2).\nUg1/Ug2: bias windings, floating on M1/M2; bias adjust P1..P6."
 		(exclude_from_sim no)
 		(at 187.96 345.44 0)
@@
 			)
 		)
-		(property "Value" "OPT PPP Rkk 330R"
+		(property "Value" "AP-634/2"
 			(at 538.48 156.718 0)
 			(effects
@@
 			)
 		)
-		(property "Description" ""
+		(property "Description" "Push-pull output transformer for PPP stages with 6x EL34 or 4x KT88"
+			(at 538.48 143.51 0)
+			(effects
+				(font
+					(size 1.27 1.27)
+				)
+				(hide yes)
+			)
+		)
+		(property "Manufacturer" "EXPERIENCE electronics"
+			(at 538.48 143.51 0)
+			(effects
+				(font
+					(size 1.27 1.27)
+				)
+				(hide yes)
+			)
+		)
+		(property "MPN" "AP-634/2"
+			(at 538.48 143.51 0)
+			(effects
+				(font
+					(size 1.27 1.27)
+				)
+				(hide yes)
+			)
+		)
+		(property "Specs" "Rkk 330Ω, >140W"
+			(at 538.48 159.512 0)
+			(effects
+				(font
+					(size 1.27 1.27)
+				)
+			)
+		)
+		(property "Secondary" "4 / 6 / 8 Ohm"
+			(at 538.48 143.51 0)
+			(effects
+				(font
+					(size 1.27 1.27)
+				)
+				(hide yes)
+			)
+		)
+		(property "Core" "MD 85 B, 85 x 102 x 75 mm, stud mounting"
+			(at 538.48 143.51 0)
+			(effects
+				(font
+					(size 1.27 1.27)
+				)
+				(hide yes)
+			)
+		)
+		(property "Frequency response" "20 Hz...20 kHz (-0.3 dB), 80 kHz (-3 dB)"
 			(at 538.48 143.51 0)
 			(effects

Commit message: KT88 variant: 4x KT88 instead of 6x EL34
- New ppp:KT88 symbol (beam tetrode, pin 1 n.c., no G3 pin)
- V3-V6 -> KT88, G3-cathode links removed
- Third output column removed (V7, V8, C13, C14, R23, R24, R29, R30,
  R35, R36, R41, R42, R47, R48, P5, P6)
- Grid leaks R19-R22 220k -> 150k (KT88 fixed-bias Rg1 max)
- Titles/notes updated, PDF regenerated
- KT88.md: feasibility analysis and open points

Co-Authored-By: Claude Opus 5.5 <noreply@anthropic.com>
Parts:
- removed C13, C14: 0.22µ/630V, Capacitor_THT:C_Rect_L26.5mm_W6.0mm_P22.50mm_MKS4, symbol Device:C
- removed P5, P6: 25k, Potentiometer_THT:Potentiometer_Piher_PT-10-V10_Vertical_Hole, symbol Device:R_Potentiometer_Trim
- removed R23, R24: 220k, Resistor_THT:R_Axial_DIN0207_L6.3mm_D2.5mm_P10.16mm_Horizontal, symbol Device:R
- removed R29, R30: 33k, Resistor_THT:R_Axial_DIN0207_L6.3mm_D2.5mm_P10.16mm_Horizontal, symbol Device:R
- removed R35, R36: 10k, Resistor_THT:R_Axial_DIN0207_L6.3mm_D2.5mm_P10.16mm_Horizontal, symbol Device:R
- removed R41, R42: 10R, Resistor_THT:R_Axial_DIN0207_L6.3mm_D2.5mm_P10.16mm_Horizontal, symbol Device:R
- removed R47, R48: 150R, Resistor_THT:R_Axial_DIN0414_L11.9mm_D4.5mm_P15.24mm_Horizontal, symbol Device:R
- removed V7, V8: EL34, Valve:Valve_Octal, symbol ppp:EL34
- R19, R20, R21, R22: value 220k -> 150k
- V3, V4, V5, V6: value EL34 -> KT88; symbol ppp:EL34 -> ppp:KT88
Connections:
- net at C6.2, R10.2, R37.1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: no longer V3.1 (G3)
- net at R40.2, V6.8 (K): no longer V6.1 (G3)
- net at R38.2, V4.8 (K): no longer V4.1 (G3)
- net at R39.1, V5.8 (K): no longer V5.1 (G3)
Other:
- note added: "Original designators: V1=Rö1 (ECC83), V2=Rö2 (ECC81), V3..V6=Rö3..Rö6 (KT88 variant, original EL34; Rö7/Rö8 omitted), T1=Ü1 (E-1220), T2=Ü2 (AP-634/2). Supply rails A1/G1/M1, A2/G2/M2 and UG1/UG2 come from the power supply sheet. Upper tubes: anode A1, screen G1, cathode M1 (G1 is referenced to M1). Lower tubes: anode A2, screen G2, cathode M2 (G2 is referenced to M2). Ug1/Ug2: bias windings, flo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"
- note added: "PPP 4x KT88 - Amplifier"
- note removed: "Original designators: V1=Rö1 (ECC83), V2=Rö2 (ECC81), V3..V8=Rö3..Rö8 (EL34), T1=Ü1 (E-1220), T2=Ü2 (AP-634/2). Supply rails A1/G1/M1, A2/G2/M2 and UG1/UG2 come from the power supply sheet. Upper tubes: anode A1, screen G1, cathode M1 (G1 is referenced to M1). Lower tubes: anode A2, screen G2, cathode M2 (G2 is referenced to M2). Ug1/Ug2: bias windings, floating on M1/M2; bias adjust P1..P6."
- note removed: "PPP 6x EL34 - Amplifier"
- title: PPP power amplifier 6x EL34 - amplifier (mono) -> PPP power amplifier 4x KT88 - amplifier (mono)
