File: supply.kicad_sch (KiCad schematic)
At the start: 14 parts, among them J101 Mains L/N/PE, SW101 Mains, T101 NTR-P/1 (mono)

Commit message: Fix bias pot wiring: grid leak resistors to pot wiper
R19..R24 now connect to the wiper (pin 2) of P1..P6; the pots form the
divider between the 33k resistors and the bias line.

Co-Authored-By: Claude Opus 5.5 <noreply@anthropic.com>
Parts:
- removed D102: B500C1500, Diode_THT:Diode_Bridge_Round_D9.0mm, symbol Device:D_Bridge_+-AA
- removed J101: Mains L/N/PE, TerminalBlock_Phoenix:TerminalBlock_Phoenix_MKDS-1,5-3_1x03_P5.00mm_Horizontal, symbol Connector_Generic:Conn_01x03
- added C102: 470µ/450V, Capacitor_THT:CP_Radial_D35.0mm_P10.00mm_SnapIn, symbol Device:C_Polarized
- added T101: NTR-P/1 (mono), symbol ppp:T_Mains_PPP
- D102: renamed from T101; value NTR-P/1 (mono) -> B500C1500; footprint (none) -> Diode_THT:Diode_Bridge_Round_D9.0mm; symbol ppp:T_Mains_PPP -> Device:D_Bridge_+-AA
- J101: renamed from C102; value 470µ/450V -> Mains L/N/PE; footprint Capacitor_THT:CP_Radial_D35.0mm_P10.00mm_SnapIn -> TerminalBlock_Phoenix:TerminalBlock_Phoenix_MKDS-1,5-3_1x03_P5.00mm_Horizontal; symbol Device:C_Polarized -> Connector_Generic:Conn_01x03
Connections:
- net A1: now also C102.1; no longer J101.1
- net A2: now also D102.1 (+)
- net Earth_Protective: now also J101.3 (Pin_3)
- net HEATER_A: now also T101.5 (S5); no longer D102.5 (S5)
- net HEATER_B: now also T101.6 (S6); no longer D102.6 (S6)
- net M1: now also D102.2 (-), T101.8 (S8); no longer D102.8 (S8)
- net M2: now also C102.2, T101.10 (S10); no longer D102.10 (S10), J101.2
- net UG1: now also T101.7 (S7); no longer D102.7 (S7)
- net UG2: now also T101.9 (S9); no longer D102.9 (S9)
- net at SW101.3: now also T101.1 (PRI1); no longer D102.1 (PRI1)
- net at SW101.1: now also T101.2 (PRI2); no longer D102.2 (PRI2)
- net at D101.3: now also T101.3 (S3); no longer D102.3 (S3)
- net at D101.4: now also T101.4 (S4); no longer D102.4 (S4)
- net at F101.2: now also J101.1 (Pin_1)
- net at SW101.2: now also J101.2 (Pin_2)
- new net: D102.3, T101.11 (S11)
- new net: D102.4, T101.12 (S12)

Commit message: KT88 variant: 4x KT88 instead of 6x EL34
- New ppp:KT88 symbol (beam tetrode, pin 1 n.c., no G3 pin)
- V3-V6 -> KT88, G3-cathode links removed
- Third output column removed (V7, V8, C13, C14, R23, R24, R29, R30,
  R35, R36, R41, R42, R47, R48, P5, P6)
- Grid leaks R19-R22 220k -> 150k (KT88 fixed-bias Rg1 max)
- Titles/notes updated, PDF regenerated
- KT88.md: feasibility analysis and open points

Co-Authored-By: Claude Opus 5.5 <noreply@anthropic.com>
Other:
- note added: "PPP 4x KT88 - Power supply"
- note removed: "PPP 6x EL34 - Power supply"
- title: PPP power amplifier 6x EL34 - power supply (mono) -> PPP power amplifier 4x KT88 - power supply (mono)
Changed lines of the file:
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@@
 	(paper "A3")
 	(title_block
-		(title "PPP power amplifier 6x EL34 - power supply (mono)")
+		(title "PPP power amplifier 4x KT88 - power supply (mono)")
 		(date "2026-10-20")
 		(rev "1")
@@
 		)
 	)
-	(text "PPP 6x EL34 - Power supply"
+	(text "PPP 4x KT88 - Power supply"
 		(exclude_from_sim no)
 		(at 50.8 50.8 0)

Commit message: KT88: 12.6V heaters, centre grounded at the tubes
- ECC83/ECC81 in 12.6V mode (pins 4-5), pin 9 to GND
- KT88 heaters in series strings V3+V4, V5+V6, midpoints to GND
- Remove hum-balance resistors R49/R50
- T101: custom transformer, 12.6V 4A heater winding (no CT),
  HV windings 310V 0.35A
- KT88.md updated

Co-Authored-By: Claude Opus 5.5 <noreply@anthropic.com>
Parts:
- T101: value NTR-P/1 (mono) -> custom (mono)
Other:
- note added: "Custom mains transformer per monoblock (replaces the NTR-P/1): 2x 310V 0.35A, 12.6V 4A (no CT). Aux windings Ug1/Ug2 added for the grid bias supplies (approx. 60V~ / 50mA, value TBD). UG1 winding floats on M1, UG2 winding floats on M2."
- note removed: "Mono half of the original stereo supply (NTR-P/1: 4x 310V, 2x 6.3V). Aux windings Ug1/Ug2 added for the grid bias supplies (approx. 60V~ / 50mA, value TBD). UG1 winding floats on M1, UG2 winding floats on M2."
Changed lines of the file:
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@@
 		)
 	)
-	(text "Mono half of the original stereo supply (NTR-P/1: 4x 310V, 2x 6.3V).\nAux windings Ug1/Ug2 added for the grid bias supplies (approx. 60V~ / 50mA, value TBD).\nUG1 winding floats on M1, UG2 winding floats on M2."
+	(text "Custom mains transformer per monoblock (replaces the NTR-P/1): 2x 310V 0.35A, 12.6V 4A (no CT).\nAux windings Ug1/Ug2 added for the grid bias supplies (approx. 60V~ / 50mA, value TBD).\nUG1 winding floats on M1, UG2 winding floats on M2."
 		(exclude_from_sim no)
 		(at 50.8 259.08 0)
@@
 			)
 		)
-		(property "Value" "NTR-P/1 (mono)"
+		(property "Value" "custom (mono)"
 			(at 254 188.468 0)
 			(effects
