File: smps/smps.kicad_sch (KiCad schematic)
At the start: 60 parts, among them J101 Mains, K1 G5LE-1, Q1 IPP60R170CFD7, Q2 IPP60R170CFD7, Q3 IPP60R170CFD7, U1 IL300, U2 2EDL23N06PJXUMA1, U3 1EDN7550B, U4 STM32G474CBTx

Commit message: cleanup
Parts:
- removed C113: 100n, symbol Device:C
- removed C3: 1n, symbol Device:C
- removed R105: 10R 1W, symbol Device:R
- added D6: 1N4148WS, Diode_SMD:D_SOD-323, symbol Diode:1N4148WS
- added Q4: 2N7002, Package_TO_SOT_SMD:SOT-23, symbol Transistor_FET:2N7002
- added R21: R, symbol Device:R
- added R22: 100R, symbol Device:R
- R1, R2: value R -> 1M
- R3: value R -> 22k
- R4: value R -> 1k3
- R6: value 1k -> 1M
Connections:
- net LLC_OC is gone; now on an unnamed net: R6.2
- net GNDPWR: now also Q4.2 (S), R21.2
- net at R6.1: now also R2.2
- net LLC_HI: now reaches R15.1, R17.2
- net +15V_PRI: now reaches K1.2
- net +15V_PRI: now also C4.1, C6.1, C7.1, C8.1, U2.1 (VDD), U3.4 (VDD), D6.1 (K)
- net at K1.5: now also Q4.3 (D)
- net PFC_POS: now reaches R19.1
- net PFC_NEG: now reaches R20.1
- net LLC_EN: now reaches U2.4 (EN/FLT)
- net at R1.1: no longer R2.2
- net LLC_LO: now reaches R16.1
- net +3V3_PRI: now reaches R17.1
- new net: Q4.1 (G), R21.1, R22.1
- new net CHARGE: R22.2
Other:
- note removed: "+15V"
- note removed: "+3V3"
- moved on the sheet: C130, C4, C5, C6, C7, C8, D3, D4, L1, L2, Q1, Q2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

Commit message: added missing wire
Connections:
- net at K1.5, Q4.3 (D): now also D6.2 (A)
Changed lines of the file:
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@@
+	)
+	(junction
+		(at 135.89 106.68)
+		(diameter 0)
+		(color 0 0 0 0)
 	)
 	(junction
@@
 	(wire
 		(pts
+			(xy 125.73 92.71) (xy 135.89 92.71)
+		)
+		(stroke
+			(width 0)
+			(type default)
+		)
+	)
+	(wire
+		(pts
 			(xy 261.62 124.46) (xy 354.33 124.46)
 		)
@@
 		)
 		(stroke
+			(width 0)
+			(type default)
+		)
+	)
+	(wire
+		(pts
+			(xy 135.89 92.71) (xy 135.89 106.68)
+		)
+		(stroke
